Commit message: genmap_demo set up, but most machines not powerful enough to run robot_pose_ekf

File: gunncs_navigation_description/urdf/os.urdf (robot description, URDF)
Before this commit: robot old-subdivision, 4 links, 3 joints
Links:
- link base_footprint: geometry visual cylinder length=0.075 radius=0.170
- link base_link: geometry 
Joints:
- joint base_to_camera: parent base_link -> base_footprint
- joint base_to_imu: parent base_link -> base_footprint
- joint base_to_right_leg: child base_footprint -> base_link; parent base_link -> base_footprint

Commit message: updated urdf for tall kinect

File: gunncs_navigation_description/urdf/os.urdf (robot description, URDF)
Before this commit: robot old-subdivision, 4 links, 3 joints
Joints:
- joint base_to_camera: origin xyz=0.09 0 0.075 -> xyz=-.23 0 .50 rpy=0 .401425728   0

Commit message: changed urdf to tall kinect

File: gunncs_navigation_description/urdf/os.urdf (robot description, URDF)
Before this commit: robot old-subdivision, 4 links, 3 joints
Links:
- added link camera_link_tall; visual box size=0.08 0.25 .04
Joints:
- added joint base_to_camera_tall: type fixed, parent base_footprint, child camera_link_tall, origin xyz=-.23 0 .50 rpy=0 .401425728   0
